File: rev 2.0/Electrolytes.kicad_sch (KiCad schematic)
At the start: 105 parts, among them J1 OLED, J2 aRGB_BREAKOUT, J3 Battery, U1 Pro Micro (nice!nano)

Commit message: drc/erc clean up
Connections:
- net rotSW-R is gone; now on net rotSW_R: D1.2 (A), MX3-0_0.2 (ROW), MX3-0_7.2 (ROW)
Changed lines of the file:
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@@
     )
   )
-  (global_label "rotSW-R" (shape input) (at 43.18 103.505 0) (fields_autoplaced)
+  (global_label "rotSW_R" (shape input) (at 43.18 103.505 0) (fields_autoplaced)
     (effects (font (size 1.27 1.27)) (justify left))
-    (property "Intersheetrefs" "${INTERSHEET_REFS}" (at 54.25 103.505 0)
+    (property "Intersheetrefs" "${INTERSHEET_REFS}" (at 53.6452 103.505 0)
       (effects (font (size 1.27 1.27)) (justify left) hide)
     )
@@
     )
   )
-  (symbol (lib_id "power:GND") (at 102.87 129.54 270) (unit 1)
-    (in_bom yes) (on_board yes) (dnp no)
-    (property "Reference" "#PWR064" (at 96.52 129.54 0)
-      (effects (font (size 1.27 1.27)) hide)
-    )
-    (property "Value" "GND" (at 99.695 129.54 90)
-      (effects (font (size 1 1)) (justify right))
-    )
-    (property "Footprint" "" (at 102.87 129.54 0)
-      (effects (font (size 1.27 1.27)) hide)
-    )
-    (property "Datasheet" "" (at 102.87 129.54 0)
-      (effects (font (size 1.27 1.27)) hide)
-    )
-    (pin "1")
-    (instances
-      (project "Chop Shop (Revival)"
-        (path "/1027873b-2f6e-41c2-9a0e-e655453de127"
-          (reference "#PWR064") (unit 1)
-        )
-      )
-      (project "Hisui"
-        (path "/68a3b41d-2fa2-4c97-892f-e2f3452d514a"
-          (reference "#PWR0101") (unit 1)
-        )
-      )
-      (project "Electrolytes"
-        (path "/79f0cd58-4c68-464d-9750-2afff68b5af5"
-          (reference "#PWR013") (unit 1)
-        )
-      )
-      (project "Phony"
-        (path "/e63e39d7-6ac0-4ffd-8aa3-1841a4541b55"
-          (reference "#PWR0121") (unit 1)
-        )
-      )
-      (project "QAZ (RP2040)"
-        (path "/ee27d19c-8dca-4ac8-a760-6dfd54d28071"
-          (reference "#PWR0104") (unit 1)
-        )
-      )
-    )
-  )
   (symbol (lib_id "power:-BATT") (at 102.87 121.92 90) (unit 1)
     (in_bom yes) (on_board yes) (dnp no)
@@
     )
   )
+  (symbol (lib_id "power:GND") (at 102.87 132.08 270) (unit 1)
+    (in_bom yes) (on_board yes) (dnp no)
+    (property "Reference" "#PWR064" (at 96.52 132.08 0)
+      (effects (font (size 1.27 1.27)) hide)
+    )
+    (property "Value" "GND" (at 99.695 132.08 90)
+      (effects (font (size 1 1)) (justify right))
+    )
+    (property "Footprint" "" (at 102.87 132.08 0)
+      (effects (font (size 1.27 1.27)) hide)
+    )
+    (property "Datasheet" "" (at 102.87 132.08 0)
+      (effects (font (size 1.27 1.27)) hide)
+    )
+    (pin "1")
+    (instances
+      (project "Chop Shop (Revival)"
+        (path "/1027873b-2f6e-41c2-9a0e-e655453de127"
+          (reference "#PWR064") (unit 1)
+        )
+      )
+      (project "Hisui"
+        (path "/68a3b41d-2fa2-4c97-892f-e2f3452d514a"
+          (reference "#PWR0101") (unit 1)
+        )
+      )
+      (project "Electrolytes"
+        (path "/79f0cd58-4c68-464d-9750-2afff68b5af5"
+          (reference "#PWR09") (unit 1)
+        )
+      )
+      (project "Phony"
+        (path "/e63e39d7-6ac0-4ffd-8aa3-1841a4541b55"
+          (reference "#PWR0121") (unit 1)
+        )
+      )
+      (project "QAZ (RP2040)"
+        (path "/ee27d19c-8dca-4ac8-a760-6dfd54d28071"
+          (reference "#PWR0104") (unit 1)
+        )
+      )
+    )
+  )
   (symbol (lib_id "Shinkai_Library:MX_Switch") (at 34.29 55.245 0) (unit 1)
     (in_bom yes) (on_board yes) (dnp no) (fields_autoplaced)
@@
     )
   )
-  (symbol (lib_id "Device:RotaryEncoder_Switch") (at 121.92 175.26 0) (unit 1)
-    (in_bom yes) (on_board yes) (dnp no)
-    (property "Reference" "RE2" (at 121.92 168.91 0)
-      (effects (font (size 1 1)))
-    )
-    (property "Value" "Rotary Encoder" (at 121.92 168.91 0)
-      (effects (font (size 1 1)) hide)
-    )
-    (property "Footprint" "PCM_marbastlib-various:ROT_Alps_EC11E-Switch" (at 118.11 171.196 0)
-      (effects (font (size 1.27 1.27)) hide)
-    )
-    (property "Datasheet" "~" (at 121.92 168.656 0)
-      (effects (font (size 1.27 1.27)) hide)
-    )
-    (pin "A")
-    (pin "B")
-    (pin "C")
-    (pin "S1")
-    (pin "S2")
-    (instances
-      (project "Chop Shop (Revival)"
-        (path "/1027873b-2f6e-41c2-9a0e-e655453de127"
-          (reference "RE2") (unit 1)
-        )
-      )
-      (project "Electrolytes"
-        (path "/79f0cd58-4c68-464d-9750-2afff68b5af5"
-          (reference "RE1") (unit 1)
-        )
-      )
-    )
-  )
-  (symbol (lib_id "power:GND") (at 102.87 132.08 270) (unit 1)
+  (symbol (lib_id "power:GND") (at 102.87 129.54 270) (unit 1)
     (in_bom yes) (on_board yes) (dnp no)
-    (property "Reference" "#PWR064" (at 96.52 132.08 0)
+    (property "Reference" "#PWR064" (at 96.52 129.54 0)
       (effects (font (size 1.27 1.27)) hide)
     )
-    (property "Value" "GND" (at 99.695 132.08 90)
+    (property "Value" "GND" (at 99.695 129.54 90)
       (effects (font (size 1 1)) (justify right))
     )
-    (property "Footprint" "" (at 102.87 132.08 0)
+    (property "Footprint" "" (at 102.87 129.54 0)
       (effects (font (size 1.27 1.27)) hide)
     )
-    (property "Datasheet" "" (at 102.87 132.08 0)
+    (property "Datasheet" "" (at 102.87 129.54 0)
       (effects (font (size 1.27 1.27)) hide)
     )
@@
       (project "Electrolytes"
         (path "/79f0cd58-4c68-464d-9750-2afff68b5af5"
-          (reference "#PWR012") (unit 1)
+          (reference "#PWR07") (unit 1)
         )
       )
@@
         )
       )
+    )
+  )
+  (symbol (lib_id "Device:RotaryEncoder_Switch") (at 121.92 175.26 0) (unit 1)
+    (in_bom yes) (on_board yes) (dnp no)
+    (property "Reference" "RE2" (at 121.92 168.91 0)
+      (effects (font (size 1 1)))
+    )
+    (property "Value" "Rotary Encoder" (at 121.92 168.91 0)
+      (effects (font (size 1 1)) hide)
+    )
+    (property "Footprint" "PCM_marbastlib-various:ROT_Alps_EC11E-Switch" (at 118.11 171.196 0)
+      (effects (font (size 1.27 1.27)) hide)
+    )
+    (property "Datasheet" "~" (at 121.92 168.656 0)
+      (effects (font (size 1.27 1.27)) hide)
+    )
+    (pin "A")
+    (pin "B")
+    (pin "C")
+    (pin "S1")
+    (pin "S2")
+    (instances
+      (project "Chop Shop (Revival)"
+        (path "/1027873b-2f6e-41c2-9a0e-e655453de127"
+          (reference "RE2") (unit 1)
+        )
+      )
+      (project "Electrolytes"
+        (path "/79f0cd58-4c68-464d-9750-2afff68b5af5"
+          (reference "RE1") (unit 1)
+        )
+      )
